Commit message: add mekamon to existing files

File: simulation_ws/src/turtlebot3_description_reduced_mesh/urdf/turtlebot3_waffle_pi.gazebo.xacro (robot description, xacro)
@@ -1,169 +1,6 @@
 <?xml version="1.0"?>
 <robot name="turtlebot3_waffle_pi_sim" xmlns:xacro="http://ros.org/wiki/xacro">
-  <xacro:arg name="laser_visual"  default="false"/>
-  <xacro:arg name="camera_visual" default="false"/>
-  <xacro:arg name="imu_visual"    default="false"/>
-  <gazebo reference="base_link">
+  <gazebo reference="body">
     <material>Gazebo/DarkGrey</material>
   </gazebo>
-  <gazebo reference="wheel_left_link">
-    <mu1>0.1</mu1>
-    <mu2>0.1</mu2>
-    <kp>500000.0</kp>
-    <kd>10.0</kd>
-    <minDepth>0.001</minDepth>
-    <maxVel>0.1</maxVel>
-    <fdir1>1 0 0</fdir1>
-    <material>Gazebo/FlatBlack</material>
-  </gazebo>
-  <gazebo reference="wheel_right_link">
-    <mu1>0.1</mu1>
-    <mu2>0.1</mu2>
-    <kp>500000.0</kp>
-    <kd>10.0</kd>
-    <minDepth>0.001</minDepth>
-    <maxVel>0.1</maxVel>
-    <fdir1>1 0 0</fdir1>
-    <material>Gazebo/FlatBlack</material>
-  </gazebo>
-  <gazebo reference="caster_back_right_link">
-    <mu1>0.1</mu1>
-    <mu2>0.1</mu2>
-    <kp>1000000.0</kp>
-    <kd>100.0</kd>
-    <minDepth>0.001</minDepth>
-    <maxVel>1.0</maxVel>
-    <material>Gazebo/FlatBlack</material>
-  </gazebo>
-  <gazebo reference="caster_back_left_link">
-    <mu1>0.1</mu1>
-    <mu2>0.1</mu2>
-    <kp>1000000.0</kp>
-    <kd>100.0</kd>
-    <minDepth>0.001</minDepth>
-    <maxVel>1.0</maxVel>
-    <material>Gazebo/FlatBlack</material>
-  </gazebo>
-  <gazebo reference="imu_link">
-    <sensor type="imu" name="imu">
-      <always_on>true</always_on>
-      <visualize>$(arg imu_visual)</visualize>
-    </sensor>
-    <material>Gazebo/Grey</material>
-  </gazebo>
-  <gazebo>
-    <plugin name="turtlebot3_waffle_pi_controller" filename="libgazebo_ros_diff_drive.so">
-      <commandTopic>cmd_vel</commandTopic>
-      <odometryTopic>odom</odometryTopic>
-      <odometryFrame>odom</odometryFrame>
-      <odometrySource>world</odometrySource>
-      <publishOdomTF>true</publishOdomTF>
-      <robotBaseFrame>base_footprint</robotBaseFrame>
-      <publishWheelTF>false</publishWheelTF>
-      <publishTf>true</publishTf>
-      <publishWheelJointState>true</publishWheelJointState>
-      <legacyMode>false</legacyMode>
-      <updateRate>30</updateRate>
-      <leftJoint>wheel_left_joint</leftJoint>
-      <rightJoint>wheel_right_joint</rightJoint>
-      <wheelSeparation>0.287</wheelSeparation>
-      <wheelDiameter>0.066</wheelDiameter>
-      <wheelAcceleration>1</wheelAcceleration>
-      <wheelTorque>10</wheelTorque>
-      <rosDebugLevel>na</rosDebugLevel>
-    </plugin>
-  </gazebo>
-  <gazebo>
-    <plugin name="imu_plugin" filename="libgazebo_ros_imu.so">
-      <alwaysOn>true</alwaysOn>
-      <bodyName>imu_link</bodyName>
-      <frameName>imu_link</frameName>
-      <topicName>imu</topicName>
-      <serviceName>imu_service</serviceName>
-      <gaussianNoise>0.0</gaussianNoise>
-      <updateRate>200</updateRate>
-      <imu>
-        <noise>
-          <type>gaussian</type>
-          <rate>
-            <mean>0.0</mean>
-            <stddev>2e-4</stddev>
-            <bias_mean>0.0000075</bias_mean>
-            <bias_stddev>0.0000008</bias_stddev>
-          </rate>
-          <accel>
-            <mean>0.0</mean>
-            <stddev>1.7e-2</stddev>
-            <bias_mean>0.1</bias_mean>
-            <bias_stddev>0.001</bias_stddev>
-          </accel>
-        </noise>
-      </imu>
-    </plugin>
-  </gazebo>
-  <gazebo reference="base_scan">
-    <material>Gazebo/FlatBlack</material>
-    <sensor type="ray" name="lds_lfcd_sensor">
-      <pose>0 0 0 0 0 0</pose>
-      <visualize>$(arg laser_visual)</visualize>
-      <update_rate>5</update_rate>
-      <ray>
-        <scan>
-          <horizontal>
-            <samples>360</samples>
-            <resolution>1</resolution>
-            <min_angle>0.0</min_angle>
-            <max_angle>6.28319</max_angle>
-          </horizontal>
-        </scan>
-        <range>
-          <min>0.120</min>
-          <max>3.5</max>
-          <resolution>0.015</resolution>
-        </range>
-        <noise>
-          <type>gaussian</type>
-          <mean>0.0</mean>
-          <stddev>0.01</stddev>
-        </noise>
-      </ray>
-      <plugin name="gazebo_ros_lds_lfcd_controller" filename="libgazebo_ros_laser.so">
-        <topicName>scan</topicName>
-        <frameName>base_scan</frameName>
-      </plugin>
-    </sensor>
-  </gazebo>
-<!--link : https://www.raspberrypi.org/documentation/hardware/camera/-->
-  <gazebo reference="camera_rgb_frame">
-    <sensor type="camera" name="Pi Camera">
-      <always_on>true</always_on>
-      <visualize>$(arg camera_visual)</visualize>
-      <camera>
-          <horizontal_fov>1.085595</horizontal_fov>
-          <image>
-              <width>640</width>
-              <height>480</height>
-              <format>R8G8B8</format>
-          </image>
-          <clip>
-              <near>0.03</near>
-              <far>100</far>
-          </clip>
-      </camera>
-      <plugin name="camera_controller" filename="libgazebo_ros_camera.so">
-        <alwaysOn>true</alwaysOn>
-        <updateRate>30.0</updateRate>
-        <cameraName>camera</cameraName>
-        <frameName>camera_rgb_optical_frame</frameName>
-        <imageTopicName>rgb/image_raw</imageTopicName>
-        <cameraInfoTopicName>rgb/camera_info</cameraInfoTopicName>
-        <hackBaseline>0.07</hackBaseline>
-        <distortionK1>0.0</distortionK1>
-        <distortionK2>0.0</distortionK2>
-        <distortionK3>0.0</distortionK3>
-        <distortionT1>0.0</distortionT1>
-        <distortionT2>0.0</distortionT2>
-      </plugin>
-    </sensor>
-  </gazebo>
 </robot>

File: simulation_ws/src/turtlebot3_description_reduced_mesh/urdf/turtlebot3_waffle_pi.urdf.xacro (robot description, xacro)
@@ -1,187 +1,248 @@
-<?xml version="1.0" ?>
-<robot name="turtlebot3_waffle_pi" xmlns:xacro="http://ros.org/wiki/xacro">
-  <xacro:include filename="$(find turtlebot3_description_reduced_mesh)/urdf/common_properties.xacro"/>
-  <xacro:include filename="$(find turtlebot3_description_reduced_mesh)/urdf/turtlebot3_waffle_pi.gazebo.xacro"/>
-  <link name="base_footprint"/>
-  <joint name="base_joint" type="fixed">
-    <parent link="base_footprint"/>
-    <child link="base_link" />
-    <origin xyz="0 0 0.010" rpy="0 0 0"/>
+<?xml version="1.0"?>
+<robot name="mekamon" xmlns:xacro="http://ros.org/wiki/xacro">
+  <!-- units are metres & Kg-->
+  <xacro:property name="body_x" value="0.115" />
+  <xacro:property name="body_y" value="0.115" />
+  <xacro:property name="body_z" value="0.075" />
+  <xacro:property name="headradius" value="0.025" />
+  <!-- all leg parts can have same width & height, just vary length -->
+  <xacro:property name="legwidth" value="0.03" />
+  <xacro:property name="legheight" value="0.03" />
+  <xacro:property name="hiplength" value="0.04" /><!-- from socket to hip joint -->
+  <xacro:property name="hiplinklength" value="0.03" /><!-- link from hip to thigh -->
+  <xacro:property name="thighlength" value="0.09" /><!-- from thigh joint to knee joint -->
+  <xacro:property name="foreleglength" value="0.105" /><!-- from knee joint to foot -->
+  <xacro:property name="footradius" value="0.02" /><!-- foot sphere -->
+  <xacro:property name="pi" value="3.1415" />
+  <material name="body">
+    <color rgba="1.0 1.0 1.0 1"/>
+  </material>
+  <material name="head">
+    <color rgba="0.1 0.1 0.9 1"/>
+  </material>
+  <material name="hip">
+    <color rgba="0.5 0.5 0.5 1"/>
+  </material>
+  <material name="hiplink">
+    <color rgba="0.1 0.1 0.1 1"/>
+  </material>
+  <material name="thigh">
+    <color rgba="0.5 0.5 0.5 1"/>
+  </material>
+  <material name="foreleg">
+    <color rgba="0.1 0.1 0.1 1"/>
+  </material>
+  <material name="foot">
+    <color rgba="0.9 0.9 0.9 0.9"/>
+  </material>
+  <!-- Standard moment of inertia tensor for solid sphere -->
+  <xacro:macro name="sphere_inertial" params="mass radius">
+    <inertial>
+      <mass value="${mass}" />
+      <inertia ixx="${0.4 * mass * radius * radius}" ixy="0.0" ixz="0.0"
+                         iyy="${0.4 * mass * radius * radius}" iyz="0.0"
+                                   izz="${0.4 * mass * radius * radius}" />
+    </inertial>
+  </xacro:macro>
+  <!-- Standard moment of inertia tensor for solid cuboid -->
+  <xacro:macro name="box_inertial" params="mass x y z">
+    <inertial>
+      <mass value="${mass}" />
+      <inertia ixx="${0.0833333 * mass * (y*y + z*z)}" ixy="0.0" ixz="0.0"
+                         iyy="${0.0833333 * mass * (x*x + z*z)}" iyz="0.0"
+                                   izz="${0.0833333 * mass * (x*x + y*y)}" />
+    </inertial>
+  </xacro:macro>
+  <!-- base coordinate frame link is not a physical object -->
+  <link name="base_link"/>
+  <!-- base link needs a fixed joint to first real link -->
+  <joint name="base_link_fixedjoint" type="fixed">
+    <parent link="base_link"/>
+    <child link="body"/>
+    <origin xyz="0.0 0.0 0.0" rpy="0.0 0.0 0.0"/>
   </joint>
-  <link name="base_link">
+  <!-- central body (first real link) -->
+  <link name="body">
     <visual>
-      <origin xyz="-0.064 0 0.0" rpy="0 0 0"/>
-      <geometry>
-        <mesh filename="package://turtlebot3_description_reduced_mesh/meshes/bases/waffle_pi_base_reduced.stl" scale="0.001 0.001 0.001"/>
-      </geometry>
-      <material name="light_black"/>
+      <geometry>
+          <box size="${body_x} ${body_y} ${body_z}"/>
+      </geometry>
+      <material name="body"/>
     </visual>
     <collision>
-      <origin xyz="-0.064 0 0.047" rpy="0 0 0"/>
-      <geometry>
-        <box size="0.266 0.266 0.094"/>
+      <geometry>
+          <box size="${body_x} ${body_y} ${body_z}"/>
       </geometry>
     </collision>
-    <inertial>
-      <origin xyz="0 0 0" rpy="0 0 0"/>
-      <mass value="1.3729096e+00"/>
-      <inertia ixx="8.7002718e-03" ixy="-4.7576583e-05" ixz="1.1160499e-04"
-               iyy="8.6195418e-03" iyz="-3.5422299e-06"
-               izz="1.4612727e-02" />
-    </inertial>
+    <xacro:box_inertial mass="0.5" x="${body_x}" y="${body_y}" z="${body_z}"/>
   </link>
-  <joint name="wheel_left_joint" type="continuous">
-    <parent link="base_link"/>
-    <child link="wheel_left_link"/>
-    <origin xyz="0.0 0.144 0.023" rpy="-1.57 0 0"/>
-    <axis xyz="0 0 1"/>
-  </joint>
-  <link name="wheel_left_link">
+  <!-- Head -->
+  <link name="head">
     <visual>
-      <origin xyz="0 0 0" rpy="1.57 0 0"/>
-      <geometry>
-        <mesh filename="package://turtlebot3_description_reduced_mesh/meshes/wheels/left_tire_reduced.stl" scale="0.001 0.001 0.001"/>
-      </geometry>
-      <material name="dark"/>
+      <geometry>
+        <sphere radius="${headradius}"/>
+      </geometry>
+      <material name="head"/>
     </visual>
     <collision>
-      <origin xyz="0 0 0" rpy="0 0 0"/>
-      <geometry>
-        <cylinder length="0.018" radius="0.033"/>
+      <geometry>
+        <sphere radius="${headradius}"/>
       </geometry>
     </collision>
-    <inertial>
-      <origin xyz="0 0 0" />
-      <mass value="2.8498940e-02" />
-      <inertia ixx="1.1175580e-05" ixy="-4.2369783e-11" ixz="-5.9381719e-09"
-               iyy="1.1192413e-05" iyz="-1.4400107e-11"
-               izz="2.0712558e-05" />
-      </inertial>
+    <xacro:sphere_inertial mass="0.01" radius="${headradius}"/>
   </link>
-  <joint name="wheel_right_joint" type="continuous">
-    <parent link="base_link"/>
-    <child link="wheel_right_link"/>
-    <origin xyz="0.0 -0.144 0.023" rpy="-1.57 0 0"/>
-    <axis xyz="0 0 1"/>
+  <!-- body-to-head static joint -->
+  <joint name="body_to_head" type="fixed">
+    <parent link="body"/>
+    <child link="head"/>
+    <origin xyz="0.03 0.00 0.04" />
   </joint>
-  <link name="wheel_right_link">
-    <visual>
-      <origin xyz="0 0 0" rpy="1.57 0 0"/>
-      <geometry>
-        <mesh filename="package://turtlebot3_description_reduced_mesh/meshes/wheels/right_tire_reduced.stl" scale="0.001 0.001 0.001"/>
-      </geometry>
-      <material name="dark"/>
-    </visual>
-    <collision>
-      <origin xyz="0 0 0" rpy="0 0 0"/>
-      <geometry>
-        <cylinder length="0.018" radius="0.033"/>
-      </geometry>
-    </collision>
-    <inertial>
-      <origin xyz="0 0 0" />
-      <mass value="2.8498940e-02" />
-      <inertia ixx="1.1175580e-05" ixy="-4.2369783e-11" ixz="-5.9381719e-09"
-               iyy="1.1192413e-05" iyz="-1.4400107e-11"
-               izz="2.0712558e-05" />
-      </inertial>
-  </link>
-  <joint name="caster_back_right_joint" type="fixed">
-    <parent link="base_link"/>
-    <child link="caster_back_right_link"/>
-    <origin xyz="-0.177 -0.064 -0.004" rpy="-1.57 0 0"/>
-  </joint>
-  <link name="caster_back_right_link">
-    <collision>
-      <origin xyz="0 0.001 0" rpy="0 0 0"/>
-      <geometry>
-        <box size="0.030 0.009 0.020"/>
-      </geometry>
-    </collision>
-    <inertial>
-      <origin xyz="0 0 0" />
-      <mass value="0.005" />
-      <inertia ixx="0.001" ixy="0.0" ixz="0.0"
-               iyy="0.001" iyz="0.0"
-               izz="0.001" />
-    </inertial>
-  </link>
-  <joint name="caster_back_left_joint" type="fixed">
-    <parent link="base_link"/>
-    <child link="caster_back_left_link"/>
-    <origin xyz="-0.177 0.064 -0.004" rpy="-1.57 0 0"/>
-  </joint>
-  <link name="caster_back_left_link">
-    <collision>
-      <origin xyz="0 0.001 0" rpy="0 0 0"/>
-      <geometry>
-        <box size="0.030 0.009 0.020"/>
-      </geometry>
-    </collision>
-    <inertial>
-      <origin xyz="0 0 0" />
-      <mass value="0.005" />
-      <inertia ixx="0.001" ixy="0.0" ixz="0.0"
-               iyy="0.001" iyz="0.0"
-               izz="0.001" />
-    </inertial>
-  </link>
-  <joint name="imu_joint" type="fixed">
-    <parent link="base_link"/>
-    <child link="imu_link"/>
-    <origin xyz="0.0 0 0.068" rpy="0 0 0"/>
-  </joint>
-  <link name="imu_link"/>
-  <joint name="scan_joint" type="fixed">
-    <parent link="base_link"/>
-    <child link="base_scan"/>
-    <origin xyz="-0.064 0 0.122" rpy="0 0 0"/>
-  </joint>
-  <link name="base_scan">
-    <visual>
-      <origin xyz="0 0 0.0" rpy="0 0 0"/>
-      <geometry>
-        <mesh filename="package://turtlebot3_description_reduced_mesh/meshes/sensors/lds.stl" scale="0.001 0.001 0.001"/>
-      </geometry>
-      <material name="dark"/>
-    </visual>
-    <collision>
-      <origin xyz="0.015 0 -0.0065" rpy="0 0 0"/>
-      <geometry>
-        <cylinder length="0.0315" radius="0.055"/>
-      </geometry>
-    </collision>
-    <inertial>
-      <mass value="0.114" />
-      <origin xyz="0 0 0" />
-      <inertia ixx="0.001" ixy="0.0" ixz="0.0"
-               iyy="0.001" iyz="0.0"
-               izz="0.001" />
-    </inertial>
-  </link>
-  <joint name="camera_joint" type="fixed">
-    <origin xyz="0.073 -0.011 0.084" rpy="0 0 0"/>
-    <parent link="base_link"/>
-    <child link="camera_link"/>
-  </joint>
-  <link name="camera_link">
-    <collision>
-      <origin xyz="0.005 0.011 0.013" rpy="0 0 0"/>
-      <geometry>
-        <box size="0.015 0.030 0.027"/>
-      </geometry>
-    </collision>
-  </link>
-  <joint name="camera_rgb_joint" type="fixed">
-    <origin xyz="0.003 0.011 0.009" rpy="0 0 0"/>
-    <parent link="camera_link"/>
-    <child link="camera_rgb_frame"/>
-  </joint>
-  <link name="camera_rgb_frame"/>
-  <joint name="camera_rgb_optical_joint" type="fixed">
-    <origin xyz="0 0 0" rpy="-1.57 0 -1.57"/>
-    <parent link="camera_rgb_frame"/>
-    <child link="camera_rgb_optical_frame"/>
-  </joint>
-  <link name="camera_rgb_optical_frame"/>
+  <!-- Leg builder macro
+  arg 'prefix' is link name prefix.
+  args 'reflect' used in leg placement. -->
+  <xacro:macro name="leg" params="prefix reflect_x reflect_y hipangle">
+    <!-- body-to-hip static joint -->
+    <joint name="body_to_${prefix}_hip" type="fixed">
+      <parent link="body"/>
+      <child link="${prefix}_hip"/>
+      <!-- Where this joint attaches to the parent link,
+      relative to previous joint origin -->
+      <origin xyz="${reflect_x*0.04} ${reflect_y*0.04} -0.025"
+              rpy="0 0 ${pi/4 + hipangle*pi/2}"/>
+    </joint>
+    <!-- Hip, containing servo -->
+    <link name="${prefix}_hip">
+      <visual>
+        <geometry>
+          <!--length, width, height-->
+          <box size="${hiplength} ${legwidth} ${legheight}"/>
+        </geometry>
+        <!-- Where we want the link centre to be, relative to the joint? -->
+        <origin xyz="${hiplength/2} 0 0" rpy="0 0 0"/>
+        <material name="hip"/>
+      </visual>
+      <collision>
+        <!--same as visual geometry -->
+        <geometry>
+          <box size="${hiplength} ${legwidth} ${legheight}"/>
+        </geometry>
+        <!--same as visual geometry -->
+        <origin xyz="${hiplength/2} 0 0" rpy="0 0 0"/>
+      </collision>
+      <xacro:box_inertial mass="0.02" x="${hiplength}" y="${legwidth}" z="${legheight}" />
+    </link>
+    <!-- hip-to-hiplink joint -->
+    <joint name="${prefix}_hip_joint" type="revolute">
+      <axis xyz="0 0 1"/>
+      <limit effort="1000.0" lower="-${pi/3}" upper="${pi/3}" velocity="0.5"/>
+      <!-- Where this joint attaches to the parent link,
+      relative to previous joint origin -->
+      <origin rpy="0 0 0" xyz="${hiplength} 0 0"/>
+      <parent link="${prefix}_hip"/>
+      <child link="${prefix}_hiplink"/>
+    </joint>
+    <!-- Hiplink - small passive right-angle link -->
+    <link name="${prefix}_hiplink">
+      <visual>
+        <geometry>
+          <box size="${hiplinklength} ${legwidth} ${legheight}"/>
+        </geometry>
+        <origin xyz="${hiplinklength/2} 0 0" rpy="0 0 0"/>
+        <material name="hiplink"/>
+      </visual>
+      <collision>
+        <geometry>
+          <box size="${hiplinklength} ${legwidth} ${legheight}"/>
+        </geometry>
+        <origin xyz="${hiplinklength/2} 0 0" rpy="0 0 0"/>
+      </collision>
+      <xacro:box_inertial mass="0.01" x="${hiplinklength}" y="${legwidth}" z="${legheight}" />
+    </link>
+    <!-- hiplink-to-thigh joint -->
+    <joint name="${prefix}_hiplink_joint" type="revolute">
+      <axis xyz="0 1 0"/>
+      <limit effort="1000.0" lower="-1.396" upper="1.484" velocity="0.5"/>
+      <!-- Where this joint attaches to the parent link,
+      relative to previous joint origin -->
+      <origin rpy="0 0 0" xyz="${hiplinklength} 0 0"/>
+      <parent link="${prefix}_hiplink"/>
+      <child link="${prefix}_thigh"/>
+    </joint>
+    <!-- Thigh -->
+    <link name="${prefix}_thigh">
+      <visual>
+        <geometry>
+          <box size="${thighlength} ${legwidth} ${legheight}"/>
+        </geometry>
+        <origin xyz="${thighlength/2} 0 0" rpy="0 0 0"/>
+        <material name="thigh"/>
+      </visual>
+      <collision>
+        <geometry>
+          <box size="${thighlength} ${legwidth} ${legheight}"/>
+        </geometry>
+        <origin xyz="${thighlength/2} 0 0" rpy="0 0 0"/>
+      </collision>
+      <xacro:box_inertial mass="0.05" x="${thighlength}" y="${legwidth}" z="${legheight}" />
+    </link>
+    <!-- Knee, thigh-to-foreleg joint -->
+    <joint name="${prefix}_knee_joint" type="revolute">
+      <axis xyz="0 1 0"/>
+      <limit effort="1000.0" lower="-1.169" upper="1.274" velocity="0.5"/>
+      <!-- Where this joint attaches to the parent link,
+      relative to previous joint origin -->
+      <origin rpy="0 0 0" xyz="${thighlength} 0 0"/>
+      <parent link="${prefix}_thigh"/>
+      <child link="${prefix}_foreleg"/>
+    </joint>
+    <!-- Foreleg -->
+    <link name="${prefix}_foreleg">
+      <visual>
+        <geometry>
+          <box size="${foreleglength} ${legwidth} ${legheight}"/>
+        </geometry>
+        <!-- translation of origin is relative to pre-rotation frame,
+        so x-trans is done as z-trans-->
+        <origin rpy="0 ${pi/2} 0" xyz="0 0 -${foreleglength/2}" />
+        <material name="foreleg"/>
+      </visual>
+      <collision>
+        <geometry>
+          <box size="${foreleglength} ${legwidth} ${legheight}"/>
+        </geometry>
+        <origin rpy="0 ${pi/2} 0" xyz="0 0 -${foreleglength/2}" />
+      </collision>
+      <xacro:box_inertial mass="0.03" x="${foreleglength}" y="${legwidth}" z="${legheight}" />
+    </link>
+    <!-- Foreleg to Foot static joint -->
+    <joint name="${prefix}_ankle" type="fixed">
+      <parent link="${prefix}_foreleg"/>
+      <child link="${prefix}_foot"/>
+      <!-- Where this joint attaches to the parent link,
+      relative to previous joint origin -->
+      <origin xyz="0 0 -${foreleglength}" rpy="0 0 0"/>
+    </joint>
+    <!-- Foot -->
+    <link name="${prefix}_foot">
+      <visual>
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